File: hardware/arduino-nano/PLACADETEMPERATURAS.kicad_pcb (KiCad board)
At the start: 2 copper layers, 43.2 x 17.8 mm, 10 parts, among them J1 Analog, J2 Digital, J3 Conn_01x05, J4 Conn_01x05, J5 Conn_01x05, J6 Conn_01x05

Commit message: Actualizacao de Esquematico
Parts:
- J4, J5, J6: footprint Connector_PinHeader_1.00mm:PinHeader_1x05_P1.00mm_Vertical -> Connector_PinHeader_2.54mm:PinHeader_1x05_P2.54mm_Vertical
- moved J6 24.2 mm to (178.7, 87.3)
- moved J5 12.2 mm to (169.8, 87.3)
- moved J4 3.39 mm to (161.0, 87.3)
- moved J3 2.54 mm to (150.8, 87.3)
Routing:
- net /D12/MISO: track 0.00 -> 105.0 mm
- net /*D5: track 0.00 -> 96.0 mm
- net /D4: track 0.00 -> 84.3 mm
- net /D8: track 0.00 -> 71.0 mm, vias 0 -> 1
- net /*D3: track 0.00 -> 69.9 mm
- net /D2: track 0.00 -> 52.2 mm
- net +5V: track 0.00 -> 51.4 mm
- net GND: track 0.00 -> 49.3 mm
Other:
- board size 43.2 x 17.8 mm -> 83.8 x 40.6 mm
